Commit message: auto_collect: add auto-servo collection, calib_solver, replays; fix fov/urdf

File: urdf/calib_robot.urdf (robot description, URDF)
Before this commit: robot m20id25_calib, 12 links, 11 joints
Links:
- link gocator_sensor: geometry collision box size=0.065 0.110 0.132; visual mesh filename=file:///workspace/meshes/Gocator_2450.dae

Commit message: refactor: calibration_pipeline 框架重构 — 模块化采集器/求解器架构
- 移除旧 Num2/, Num2_common/, handeye_sim/, new_method/, common/ 目录
- 新增 calibration_pipeline/ 模块化框架（registry 注册表驱动）
- 新增 8 求解器：12dof_v2/cross/9dof/hybrid/iterative/paper1/lm_9dof/lm_6dof
- 新增 3 采集器：preset_joints/single_shot/manual
- 新增种子采集节点 seed_collection_node.py（蠕动伺服+星形路径 v30）
- 新增文档 v4/v5 版本（Phase 0a/0b/0c/1/2 完整流程）
- 新增测试框架 tests/ 及 CI 脚本
- 重构场景发布/配置/URDF 生成
- 更新 .devcontainer/docker 配置

File: urdf/calib_robot.urdf (robot description, URDF)
Before this commit: robot m20id25_calib, 12 links, 11 joints
Joints:
- joint J1_joint: limit lower=-185 upper=185 effort=7000 velocity=210 -> lower=-3.228859116 upper=3.228859116 effort=7000 velocity=3.665191429
- joint J2_joint: limit lower=-100 upper=160 effort=8000 velocity=210 -> lower=-1.745329252 upper=2.792526803 effort=8000 velocity=3.665191429
- joint J3_joint: limit lower=-90 upper=220 effort=4000 velocity=265 -> lower=-1.570796327 upper=3.839724354 effort=4000 velocity=4.625122518
- joint J4_joint: limit lower=-200 upper=200 effort=300 velocity=420 -> lower=-3.490658504 upper=3.490658504 effort=300 velocity=7.330382858
- joint J5_joint: limit lower=-179.999 upper=179.999 effort=300 velocity=420 -> lower=-3.141575200 upper=3.141575200 effort=300 velocity=7.330382858
- joint J6_joint: limit lower=-450 upper=450 effort=200 velocity=720 -> lower=-7.853981634 upper=7.853981634 effort=200 velocity=12.566370614

Commit message: 重构了项目结构，并开展了真机实验。

File: urdf/calib_robot.urdf (robot description, URDF)
Before this commit: robot m20id25_calib, 12 links, 11 joints
Links:
- added link tool0
- added link weld_gun; collision mesh filename=file:///workspace/meshes/weldgun.stl scale=0.001 0.001 0.001; visual mesh filename=file:///workspace/meshes/weldgun.stl scale=0.001 0.001 0.001
Joints:
- added joint fanuc_flange-tool0_joint: type fixed, parent fanuc_flange, child tool0, origin xyz=-0.046256 -0.000142 0.375235 rpy=-3.141540 -0.384130 -0.000070
- added joint fanuc_flange-weld_gun_joint: type fixed, parent fanuc_flange, child weld_gun, origin xyz=-0.046256 -0.000142 0.375235 rpy=-3.141540 -0.384130 -0.000070
